Commit message: final draft

File: controllers/grocery_shopper/old_good/tiago_urdf.urdf (robot description, URDF)
Before this commit: robot TIAGo Steel, 64 links, 63 joints
Links:
- added link plastic crate; collision box size=0.021 0.193 0.372; collision box size=0.021 0.193 0.372
Joints:
- added joint base_link_plastic crate_joint: type fixed, parent base_link, child plastic crate, origin xyz=0.272 -0.010001 0.236 rpy=1.570798 -0.000005 1.570798
- joint base_link_plastic crate(1)_joint: origin xyz=0.372 -0.01 0.236 rpy=1.570791 -0.000005 -3.141587 -> xyz=0.272 -0.010001 0.236 rpy=1.570798 -0.000005 1.570798
