Commit message: adding change

File: controllers/grocery_shopper/tiago_urdf.urdf (robot description, URDF)
Before this commit: robot TIAGo Steel, 65 links, 64 joints
Joints:
- joint arm_4_joint: origin xyz=-0.02 -0.027 -0.2197 rpy=1.570909 -1.5318 3.141483 -> xyz=-0.02 -0.027 -0.2197 rpy=1.570909 -1.531801 3.141483

Commit message: cleaning

File: controllers/grocery_shopper/tiago_urdf.urdf (robot description, URDF)
Before this commit: robot TIAGo Steel, 64 links, 63 joints
Links:
- added link slam_lidar_0; collision box size=0.05 0.07 0.05; visual box size=0.05 0.07 0.05
- added link slam_lidar_1; collision box size=0.05 0.07 0.05; visual box size=0.05 0.07 0.05
Joints:
- added joint base_link_slam_lidar_0_joint: type fixed, parent base_link, child slam_lidar_0, origin xyz=0.202 0 7.996 rpy=0 0 0
- added joint base_link_slam_lidar_1_joint: type fixed, parent base_link, child slam_lidar_1, origin xyz=0.202 0 7.996 rpy=0 0 3.14159
- joint CASTER_WHEEL_BACK_LEFT_JOINT: origin xyz=-0.1735 0.102 -0.0335 rpy=0 0.000001 -0.08667 -> xyz=-0.1735 0.102 -0.0335 rpy=0 0.000001 0.762229
- joint CASTER_WHEEL_BACK_RIGHT_JOINT: origin xyz=-0.1735 -0.102 -0.0335 rpy=0 0.000003 -0.120633 -> xyz=-0.1735 -0.102 -0.0335 rpy=0 0.000003 -0.833131
- joint CASTER_WHEEL_FRONT_LEFT_JOINT: origin xyz=0.1695 0.102 -0.0335 rpy=0 0.000003 -0.14025 -> xyz=0.1695 0.102 -0.0335 rpy=0 0.000003 -0.264625
- joint CASTER_WHEEL_FRONT_RIGHT_JOINT: origin xyz=0.1695 -0.102 -0.0335 rpy=0 0.000005 -0.173648 -> xyz=0.1695 -0.102 -0.0335 rpy=0 0.000005 -0.331093
- joint SMALL_WHEEL_JOINT: origin xyz=-0.016001 0.000001 -0.03983 rpy=-1.5708 0.044384 0 -> xyz=-0.016001 0.000001 -0.03983 rpy=-1.5708 0.019738 0
- joint SMALL_WHEEL_JOINT_0: origin xyz=-0.016004 0.000002 -0.039547 rpy=-1.5708 0.035051 0 -> xyz=-0.016004 0.000002 -0.039547 rpy=-1.5708 0.060546 0
- joint SMALL_WHEEL_JOINT_1: origin xyz=-0.016004 0.000002 -0.03954 rpy=-1.5708 0.046738 0 -> xyz=-0.016004 0.000002 -0.03954 rpy=-1.5708 0.04558 0
- joint SMALL_WHEEL_JOINT_2: origin xyz=-0.016007 0.000003 -0.039257 rpy=-1.5708 0.037623 0 -> xyz=-0.016007 0.000003 -0.039257 rpy=-1.5708 0.031918 0
- joint arm_1_joint: origin xyz=0.025 0.194 -0.16 rpy=0 0 0.008881 -> xyz=0.025 0.194 -0.16 rpy=0 0 0.008882
- joint arm_2_joint: origin xyz=0.1251 0.019499 -0.042 rpy=1.5708 0.000023 0 -> xyz=0.1251 0.019499 -0.042 rpy=1.5708 0.000056 0
- joint arm_4_joint: origin xyz=-0.02 -0.027 -0.2197 rpy=1.570909 -1.531801 3.141483 -> xyz=-0.02 -0.027 -0.2197 rpy=1.570909 -1.531814 3.141483
- joint arm_5_joint: origin xyz=-0.162025 0.019922 0.027 rpy=-1.570797 -0.250796 1.5708 -> xyz=-0.162025 0.019922 0.027 rpy=-1.570797 -0.251226 1.5708
- joint arm_6_joint: origin xyz=0 0 0.15 rpy=2.269806 -1.570792 2.44258 -> xyz=0 0 0.15 rpy=2.05401 -1.57079 2.658376
- joint base_link_base_cover_link_joint: origin xyz=0 0 0.029988 rpy=0 0 0 -> xyz=0.000001 -0.000001 0.029976 rpy=0 0 0
- joint front_cap screw(19)_joint: origin xyz=0.049882 -0.002899 -0.0004 rpy=3.14159 0 0 -> xyz=0.086502 -0.002896 -0.0004 rpy=3.14159 0 0
- joint gripper_left_finger_joint: limit lower=0 upper=0.045 effort=16 velocity=0.05 -> lower=0 upper=0.0450018 effort=16 velocity=0.05; origin xyz=0.008365 0 0 rpy=0 0 3.1415 -> xyz=-0.000001 0 0 rpy=0 0 3.1415
- joint gripper_right_finger_joint: limit lower=0 upper=0.045 effort=16 velocity=0.05 -> lower=-9.63949e-07 upper=0.045 effort=16 velocity=0.05
- joint head_1_joint: origin xyz=0.182 0 -0.000254 rpy=-0.000004 0 -1.570796 -> xyz=0.182 0 -0.000254 rpy=-0.000004 0 -1.570795
- joint head_2_joint: axis 0 0.000004 1 -> -1 0.000005 -0.000002; origin xyz=0.005002 0.000026 0.097981 rpy=1.5708 0 0 -> xyz=0.005002 0.000026 0.097981 rpy=1.570798 -0.000005 1.570798
- joint head_2_link_display_joint: origin xyz=0.107 0.06019 -0.000001 rpy=0 0 0 -> xyz=0.107003 0.060011 0.000007 rpy=0 0 0
- joint wheel_left_joint: origin xyz=0 0.2022 0 rpy=1.570801 0.015623 0 -> xyz=0 0.2022 0 rpy=1.570801 0.015687 0
- joint wheel_right_joint: origin xyz=-0.000002 -0.202145 0.000193 rpy=1.570801 0.015525 0 -> xyz=-0.000002 -0.202145 0.000193 rpy=1.570801 0.015425 0
